Commit message: Combined spot arm and spot body into one urdf

File: spot_description/urdf/spot.urdf.xacro (robot description, xacro)
@@ -13,5 +13,4 @@
         </collision>
     </link>
-    <link name="base_link"/>
     <joint name="base_link_joint" type="fixed">
         <origin xyz="0 0 0" rpy="0 0 0" />
@@ -261,4 +260,6 @@
     <!-- Standard accessories. -->
     <xacro:include filename="$(find spot_description)/urdf/accessories.urdf.xacro" />
+    <!-- Spot Arm Include -->
+    <xacro:include filename="$(find spot_arm_description)/urdf/spot_arm.xacro" />
     <!-- Optional custom includes. -->
     <xacro:include filename="$(optenv SPOT_URDF_EXTRAS empty.urdf)" />
