Commit message: merged the arm and body urdfs in a better way - changed arm base frame to arm_base_link - created a joint between arm_base_link and body - deleted hardcoded import of arm urdf, use SPOT_URDF_EXTRAS now

File: Spot-Arm/spot_arm_description/urdf/spot_arm.xacro (robot description, xacro)
@@ -4,5 +4,5 @@
 <xacro:include filename="$(find spot_arm_description)/urdf/spot_arm.trans" />
 <xacro:include filename="$(find spot_arm_description)/urdf/spot_arm.gazebo" />
-<link name="base_link">
+<link name="arm_base_link">
   <inertial>
     <origin rpy="0 0 0" xyz="1.2371844231029972e-17 0.0 0.0325"/>

File: spot_description/urdf/spot.urdf.xacro (robot description, xacro)
@@ -18,4 +18,10 @@
         <child link="base_link" />
     </joint>
+    <link name="base_link" />
+    <joint name="arm_base_link_joint" type="fixed">
+        <origin xyz="0 0 0" rpy="0 0 0" />
+        <parent link="body" />
+        <child link="arm_base_link" />
+    </joint>
     <link name="front_rail"/>
     <joint name="front_rail_joint" type="fixed">
@@ -260,6 +266,4 @@
     <!-- Standard accessories. -->
     <xacro:include filename="$(find spot_description)/urdf/accessories.urdf.xacro" />
-    <!-- Spot Arm Include -->
-    <xacro:include filename="$(find spot_arm_description)/urdf/spot_arm.xacro" />
     <!-- Optional custom includes. -->
     <xacro:include filename="$(optenv SPOT_URDF_EXTRAS empty.urdf)" />

Commit message: Finished incorporating arm mesh with spot

File: Spot-Arm/spot_arm_description/urdf/spot_arm.xacro (robot description, xacro)
@@ -172,5 +172,5 @@
 </joint>
 <joint name="Joint2" type="revolute">
-  <origin rpy="0 0 0" xyz="0.015 0.0 0.05"/>
+  <origin rpy="0 3.141 0" xyz="-0.015 0.0 0.05"/>
   <parent link="link1"/>
   <child link="link2"/>

File: spot_description/urdf/spot.urdf.xacro (robot description, xacro)
@@ -20,6 +20,6 @@
     <link name="base_link" />
     <joint name="arm_base_link_joint" type="fixed">
-        <origin xyz="0 0 0" rpy="0 0 0" />
-        <parent link="body" />
+        <origin xyz="0 0 0" rpy="0 0 -1.5707" />
+        <parent link="front_rail" />
         <child link="arm_base_link" />
     </joint>
@@ -266,4 +266,6 @@
     <!-- Standard accessories. -->
     <xacro:include filename="$(find spot_description)/urdf/accessories.urdf.xacro" />
+    <!-- Spot Arm Include -->
+    <xacro:include filename="$(find spot_arm_description)/urdf/spot_arm.xacro" />
     <!-- Optional custom includes. -->
     <xacro:include filename="$(optenv SPOT_URDF_EXTRAS empty.urdf)" />

Commit message: Finished incorporating arm mesh with spot, fixed joint state publishers

File: Spot-Arm/spot_arm_description/urdf/spot_arm.xacro (robot description, xacro)
@@ -165,6 +165,6 @@
 </link>
 <joint name="Joint1" type="revolute">
-  <origin rpy="0 0 0" xyz="0.0 0.0 0.065"/>
-  <parent link="base_link"/>
+  <origin rpy="0 0 0" xyz="0 0.0 0.065"/>
+  <parent link="arm_base_link"/>
   <child link="link1"/>
   <axis xyz="0.0 0.0 1.0"/>

Commit message: Started testing spot manipulation

File: Spot-Arm/spot_arm_description/urdf/spot_arm.xacro (robot description, xacro)
@@ -175,5 +175,5 @@
   <parent link="link1"/>
   <child link="link2"/>
-  <axis xyz="-1.0 0.0 0.0"/>
+  <axis xyz="1.0 0.0 0.0"/>
   <limit effort="100" lower="-3.665191" upper="0.0" velocity="100"/>
 </joint>
